Commit message: Added gazebo simulation

File: src/arduinobot_description/urdf/arduinobot.urdf.xacro (robot description, xacro)
@@ -4,6 +4,15 @@
     <xacro:property name="effort" value="30.0" />
     <xacro:property name="velocity" value="10.0" />
+    <xacro:macro name="default_inertial" params="mass">
+        <inertial>
+            <mass value="${mass}" />
+            <inertia ixx="1.0" ixy="0.0" ixz="0.0"
+                iyy="1.0" iyz="0.0"
+                izz="1.0" />
+        </inertial>
+    </xacro:macro>
     <link name="world" />
     <link name="base_link">
+        <xacro:default_inertial mass="1.0"/>
         <visual>
             <origin rpy="0 0 0 " xyz="-0.5 -0.5 0" />
@@ -13,4 +22,11 @@
             </geometry>
         </visual>
+        <collision>
+            <origin rpy="0 0 0 " xyz="-0.5 -0.5 0" />
+            <geometry>
+                <mesh filename="package://arduinobot_description/meshes/basement.STL"
+                    scale="0.01 0.01 0.01" />
+            </geometry>
+        </collision>
     </link>
     <joint name="virtual_joint" type="fixed">
@@ -20,4 +36,5 @@
     </joint>
     <link name="base_plate">
+        <xacro:default_inertial mass="0.1" />
         <visual>
             <origin rpy="0 0 0" xyz="-0.39 -0.39 -0.56" />
@@ -27,4 +44,11 @@
             </geometry>
         </visual>
+        <collision>
+            <origin rpy="0 0 0" xyz="-0.39 -0.39 -0.56" />
+            <geometry>
+                <mesh filename="package://arduinobot_description/meshes/base_plate.STL"
+                    scale="0.01 0.01 0.01" />
+            </geometry>
+        </collision>
     </link>
     <joint name="joint1" type="revolute">
@@ -36,4 +60,5 @@
     </joint>
     <link name="forward_drive_arm">
+        <xacro:default_inertial mass="0.1" />
         <visual>
             <origin rpy="0 -${PI/2} ${PI/2}" xyz="0.19 0.06 -0.08" />
@@ -42,4 +67,11 @@
             </geometry>
         </visual>
+        <collision>
+            <origin rpy="0 -${PI/2} ${PI/2}" xyz="0.19 0.06 -0.08" />
+            <geometry>
+                <mesh filename="package://arduinobot_description/meshes/forward_drive_arm.STL"
+                    scale="0.01 0.01 0.01" />
+            </geometry>
+        </collision>
     </link>
     <joint name="joint2" type="revolute">
@@ -51,4 +83,5 @@
     </joint>
     <link name="horizontal_arm">
+        <xacro:default_inertial mass="0.1" />
         <visual>
             <origin rpy="${PI/2} 0 ${PI/2}" xyz="-0.03 -0.4 -0.06" />
@@ -57,4 +90,11 @@
             </geometry>
         </visual>
+        <collision>
+            <origin rpy="${PI/2} 0 ${PI/2}" xyz="-0.03 -0.4 -0.06" />
+            <geometry>
+                <mesh filename="package://arduinobot_description/meshes/horizontal_arm.STL"
+                    scale="0.01 0.01 0.01" />
+            </geometry>
+        </collision>
     </link>
     <joint name="joint3" type="revolute">
@@ -66,4 +106,5 @@
     </joint>
     <link name="claw_support">
+        <xacro:default_inertial mass="0.05" />
         <visual>
             <origin rpy="0 0 ${PI/2}" xyz="0 -0.05 -0.15" />
@@ -72,4 +113,11 @@
             </geometry>
         </visual>
+        <collision>
+            <origin rpy="0 0 ${PI/2}" xyz="0 -0.05 -0.15" />
+            <geometry>
+                <mesh filename="package://arduinobot_description/meshes/claw_support.STL"
+                    scale="0.01 0.01 0.01" />
+            </geometry>
+        </collision>
     </link>
     <joint name="horizontal_arm_to_claw_support" type="fixed">
@@ -79,4 +127,5 @@
     </joint>
     <link name="gripper_right">
+        <xacro:default_inertial mass="0.01" />
         <visual>
             <origin rpy="0 0 -${PI/2}" xyz="-0.1 0.5 -0.1" />
@@ -86,6 +135,14 @@
             </geometry>
         </visual>
+        <collision>
+            <origin rpy="0 0 -${PI/2}" xyz="-0.1 0.5 -0.1" />
+            <geometry>
+                <mesh filename="package://arduinobot_description/meshes/right_finger.STL"
+                    scale="0.01 0.01 0.01" />
+            </geometry>
+        </collision>
     </link>
     <link name="gripper_left">
+        <xacro:default_inertial mass="0.01" />
         <visual>
             <origin rpy="0 0 -${PI/2}" xyz="-0.04 0.5 -0.1" />
@@ -95,4 +152,11 @@
             </geometry>
         </visual>
+        <collision>
+            <origin rpy="0 0 -${PI/2}" xyz="-0.04 0.5 -0.1" />
+            <geometry>
+                <mesh filename="package://arduinobot_description/meshes/left_finger.STL"
+                    scale="0.01 0.01 0.01" />
+            </geometry>
+        </collision>
     </link>
     <joint name="joint_4" type="revolute">

Commit message: added robot controller yaml file

File: src/arduinobot_description/urdf/arduinobot.urdf.xacro (robot description, xacro)
@@ -1,4 +1,6 @@
 <?xml version="1.0"?>
 <robot xmlns:xacro="http://www.ros.org/wiki/xacro" name="arduinobot">
+    <xacro:include filename="$(find arduinobot_description)/urdf/arduinobot_gazebo.xacro"/>
+    <xacro:include filename="$(find arduinobot_description)/urdf/arduinobot_ros2_control.xacro" />
     <xacro:property name="PI" value="3.14159" />
     <xacro:property name="effort" value="30.0" />
@@ -12,7 +14,16 @@
         </inertial>
     </xacro:macro>
+    <xacro:macro name="default_transmission" params="number">
+        <transmission name="transmission_${number}">
+            <plugin>transmissiona_interface/SimpleTransmission</plugin>
+            <actuator name="motor_${number}" role="actuator1" />
+            <joint name="joine_${number}" role="joint1">
+                <mechanical_reduction>1.0</mechanical_reduction>
+            </joint>
+        </transmission>
+    </xacro:macro>
     <link name="world" />
     <link name="base_link">
-        <xacro:default_inertial mass="1.0"/>
+        <xacro:default_inertial mass="1.0" />
         <visual>
             <origin rpy="0 0 0 " xyz="-0.5 -0.5 0" />
@@ -52,5 +63,5 @@
         </collision>
     </link>
-    <joint name="joint1" type="revolute">
+    <joint name="joint_1" type="revolute">
         <parent link="base_link" />
         <child link="base_plate" />
@@ -64,5 +75,6 @@
             <origin rpy="0 -${PI/2} ${PI/2}" xyz="0.19 0.06 -0.08" />
             <geometry>
-                <mesh filename="package://arduinobot_description/meshes/forward_drive_arm.STL" scale="0.01 0.01 0.01" />
+                <mesh filename="package://arduinobot_description/meshes/forward_drive_arm.STL"
+                    scale="0.01 0.01 0.01" />
             </geometry>
         </visual>
@@ -75,5 +87,5 @@
         </collision>
     </link>
-    <joint name="joint2" type="revolute">
+    <joint name="joint_2" type="revolute">
         <parent link="base_plate" />
         <child link="forward_drive_arm" />
@@ -87,5 +99,6 @@
             <origin rpy="${PI/2} 0 ${PI/2}" xyz="-0.03 -0.4 -0.06" />
             <geometry>
-                <mesh filename="package://arduinobot_description/meshes/horizontal_arm.STL" scale="0.01 0.01 0.01" />
+                <mesh filename="package://arduinobot_description/meshes/horizontal_arm.STL"
+                    scale="0.01 0.01 0.01" />
             </geometry>
         </visual>
@@ -98,5 +111,5 @@
         </collision>
     </link>
-    <joint name="joint3" type="revolute">
+    <joint name="joint_3" type="revolute">
         <parent link="forward_drive_arm" />
         <child link="horizontal_arm" />
@@ -110,5 +123,6 @@
             <origin rpy="0 0 ${PI/2}" xyz="0 -0.05 -0.15" />
             <geometry>
-                <mesh filename="package://arduinobot_description/meshes/claw_support.STL" scale="0.01 0.01 0.01" />
+                <mesh filename="package://arduinobot_description/meshes/claw_support.STL"
+                    scale="0.01 0.01 0.01" />
             </geometry>
         </visual>
@@ -172,6 +186,10 @@
         <axis xyz="0 0 1" />
         <origin rpy="0 0 0" xyz="-0.22 0.13 -0.1" />
-        <mimic joint="joint_4" multiplier="-1"/>
+        <mimic joint="joint_4" multiplier="-1" />
         <limit lower="0.0" upper="${PI/2}" effort="${effort}" velocity="${velocity}" />
     </joint>
+    <xacro:default_transmission number="1" />
+    <xacro:default_transmission number="2" />
+    <xacro:default_transmission number="3" />
+    <xacro:default_transmission number="4" />
 </robot>
